Commit message: added atv and other dae's

File: bme_ros2_navigation/urdf/mogi_bot.urdf (robot description, URDF)
Before this commit: robot mogi_bot, 8 links, 7 joints
Links:
- link base_link: geometry collision box size=.4 .2 .1; collision sphere radius=0.0499

Commit message: chnaged wheel model

File: bme_ros2_navigation/urdf/mogi_bot.urdf (robot description, URDF)
Before this commit: robot mogi_bot, 8 links, 7 joints
Links:
- link left_wheel: geometry collision cylinder length=.05 radius=.1; visual mesh filename=package://bme_ros2_navigation/meshes/ATV_Wheel.dae
- link right_wheel: geometry collision cylinder length=.05 radius=.1; visual mesh filename=package://bme_ros2_navigation/meshes/ATV_Wheel.dae

Commit message: changed wheel back

File: bme_ros2_navigation/urdf/mogi_bot.urdf (robot description, URDF)
Before this commit: robot mogi_bot, 8 links, 7 joints
Links:
- link left_wheel: geometry collision cylinder length=.05 radius=.1; visual mesh filename=package://bme_ros2_navigation/meshes/wheel.dae
- link right_wheel: geometry collision cylinder length=.05 radius=.1; visual mesh filename=package://bme_ros2_navigation/meshes/wheel.dae

Commit message: added rear wheel tags to gazebo and urdf

File: bme_ros2_navigation/urdf/mogi_bot.urdf (robot description, URDF)
Before this commit: robot mogi_bot, 8 links, 7 joints
Links:
- added link left_rear_wheel, mass 5.0; collision cylinder length=.05 radius=.1; visual mesh filename=package://bme_ros2_navigation/meshes/wheel.dae
- added link right_rear_wheel, mass 5.0; collision cylinder length=.05 radius=.1; visual mesh filename=package://bme_ros2_navigation/meshes/wheel.dae
Joints:
- added joint left_rear_wheel_joint: type continuous, parent base_link, child left_rear_wheel, origin xyz=-0.3 0.15 0 rpy=0 0 0, axis 0 1 0, limit effort=100 velocity=10
- added joint right_rear_wheel_joint: type continuous, parent base_link, child right_rear_wheel, origin xyz=-0.3 -0.15 0 rpy=0 0 0, axis 0 1 0, limit effort=100 velocity=10

Commit message: moved front wheels 0.3 on x

File: bme_ros2_navigation/urdf/mogi_bot.urdf (robot description, URDF)
Before this commit: robot mogi_bot, 10 links, 9 joints
Joints:
- joint left_wheel_joint: origin xyz=0 0.15 0 rpy=0 0 0 -> xyz=0.3 0.15 0 rpy=0 0 0
- joint right_wheel_joint: origin xyz=0 -0.15 0 rpy=0 0 0 -> xyz=0.3 -0.15 0 rpy=0 0 0

Commit message: moved camera up z axis

File: bme_ros2_navigation/urdf/mogi_bot.urdf (robot description, URDF)
Before this commit: robot mogi_bot, 10 links, 9 joints
Joints:
- joint camera_joint: origin xyz=0.225 0 0.075 rpy=0 0 0 -> xyz=0.225 0 0.1 rpy=0 0 0

Commit message: moved cam up again

File: bme_ros2_navigation/urdf/mogi_bot.urdf (robot description, URDF)
Before this commit: robot mogi_bot, 10 links, 9 joints
Joints:
- joint camera_joint: origin xyz=0.225 0 0.1 rpy=0 0 0 -> xyz=0.225 0 0.2 rpy=0 0 0

Commit message: doubled wheel sizes and moved cam up again

File: bme_ros2_navigation/urdf/mogi_bot.urdf (robot description, URDF)
Before this commit: robot mogi_bot, 10 links, 9 joints
Links:
- link left_rear_wheel: geometry collision cylinder length=.05 radius=.1; visual mesh filename=package://bme_ros2_navigation/meshes/wheel.dae scale=2 2 2
- link left_wheel: geometry collision cylinder length=.05 radius=.1; visual mesh filename=package://bme_ros2_navigation/meshes/wheel.dae scale=2 2 2
- link right_rear_wheel: geometry collision cylinder length=.05 radius=.1; visual mesh filename=package://bme_ros2_navigation/meshes/wheel.dae scale=2 2 2
- link right_wheel: geometry collision cylinder length=.05 radius=.1; visual mesh filename=package://bme_ros2_navigation/meshes/wheel.dae scale=2 2 2
Joints:
- joint camera_joint: origin xyz=0.225 0 0.2 rpy=0 0 0 -> xyz=0.225 0 0.25 rpy=0 0 0

Commit message: decreased wheel size

File: bme_ros2_navigation/urdf/mogi_bot.urdf (robot description, URDF)
Before this commit: robot mogi_bot, 10 links, 9 joints
Links:
- link left_rear_wheel: geometry collision cylinder length=.05 radius=.1; visual mesh filename=package://bme_ros2_navigation/meshes/wheel.dae scale=1.5 1.5 1.5
- link left_wheel: geometry collision cylinder length=.05 radius=.1; visual mesh filename=package://bme_ros2_navigation/meshes/wheel.dae scale=1.5 1.5 1.5
- link right_rear_wheel: geometry collision cylinder length=.05 radius=.1; visual mesh filename=package://bme_ros2_navigation/meshes/wheel.dae scale=1.5 1.5 1.5
- link right_wheel: geometry collision cylinder length=.05 radius=.1; visual mesh filename=package://bme_ros2_navigation/meshes/wheel.dae scale=1.5 1.5 1.5

Commit message: decreased wheel size

File: bme_ros2_navigation/urdf/mogi_bot.urdf (robot description, URDF)
Before this commit: robot mogi_bot, 10 links, 9 joints
Links:
- link left_rear_wheel: geometry collision cylinder length=.05 radius=.1; visual mesh filename=package://bme_ros2_navigation/meshes/wheel.dae scale=1 1 1
- link left_wheel: geometry collision cylinder length=.05 radius=.1; visual mesh filename=package://bme_ros2_navigation/meshes/wheel.dae scale=1 1 1
- link right_rear_wheel: geometry collision cylinder length=.05 radius=.1; visual mesh filename=package://bme_ros2_navigation/meshes/wheel.dae scale=1 1 1
- link right_wheel: geometry collision cylinder length=.05 radius=.1; visual mesh filename=package://bme_ros2_navigation/meshes/wheel.dae scale=1 1 1

Commit message: wheel size 1.5, increased cam y

File: bme_ros2_navigation/urdf/mogi_bot.urdf (robot description, URDF)
Before this commit: robot mogi_bot, 10 links, 9 joints
Links:
- link left_rear_wheel: geometry collision cylinder length=.05 radius=.1; visual mesh filename=package://bme_ros2_navigation/meshes/wheel.dae scale=1.5 1.5 1.5
- link left_wheel: geometry collision cylinder length=.05 radius=.1; visual mesh filename=package://bme_ros2_navigation/meshes/wheel.dae scale=1.5 1.5 1.5
- link right_rear_wheel: geometry collision cylinder length=.05 radius=.1; visual mesh filename=package://bme_ros2_navigation/meshes/wheel.dae scale=1.5 1.5 1.5
- link right_wheel: geometry collision cylinder length=.05 radius=.1; visual mesh filename=package://bme_ros2_navigation/meshes/wheel.dae scale=1.5 1.5 1.5
Joints:
- joint camera_joint: origin xyz=0.225 0 0.25 rpy=0 0 0 -> xyz=0.225 0 0.33 rpy=0 0 0

Commit message: -wheelsize

File: bme_ros2_navigation/urdf/mogi_bot.urdf (robot description, URDF)
Before this commit: robot mogi_bot, 10 links, 9 joints
Links:
- link left_rear_wheel: geometry collision cylinder length=.05 radius=.1; visual mesh filename=package://bme_ros2_navigation/meshes/wheel.dae scale=1.25 1.25 1.25
- link left_wheel: geometry collision cylinder length=.05 radius=.1; visual mesh filename=package://bme_ros2_navigation/meshes/wheel.dae scale=1.25 1.25 1.25
- link right_rear_wheel: geometry collision cylinder length=.05 radius=.1; visual mesh filename=package://bme_ros2_navigation/meshes/wheel.dae scale=1.25 1.25 1.25
- link right_wheel: geometry collision cylinder length=.05 radius=.1; visual mesh filename=package://bme_ros2_navigation/meshes/wheel.dae scale=1.25 1.25 1.25

Commit message: -0.10 wheel size [1.15]

File: bme_ros2_navigation/urdf/mogi_bot.urdf (robot description, URDF)
Before this commit: robot mogi_bot, 10 links, 9 joints
Links:
- link left_rear_wheel: geometry collision cylinder length=.05 radius=.1; visual mesh filename=package://bme_ros2_navigation/meshes/wheel.dae scale=1.15 1.15 1.15
- link left_wheel: geometry collision cylinder length=.05 radius=.1; visual mesh filename=package://bme_ros2_navigation/meshes/wheel.dae scale=1.15 1.15 1.15
- link right_rear_wheel: geometry collision cylinder length=.05 radius=.1; visual mesh filename=package://bme_ros2_navigation/meshes/wheel.dae scale=1.15 1.15 1.15
- link right_wheel: geometry collision cylinder length=.05 radius=.1; visual mesh filename=package://bme_ros2_navigation/meshes/wheel.dae scale=1.15 1.15 1.15

Commit message: Changes applied to all wheels: Fixed RPY to 0 1.5708 0 so the wheel rotates correctly around its own axis instead of wobbling.
Kept visual origin Z offset at 0.025 so the mesh doesn’t clip into the ground.

Increased joint damping to 5.0 to stop "orbiting" or rising/falling oscillations.

Standardized axis to 0 1 0 without extra RPY on the axis itself.

File: bme_ros2_navigation/urdf/mogi_bot.urdf (robot description, URDF)
Before this commit: robot mogi_bot, 10 links, 9 joints
Links:
- link left_rear_wheel: geometry collision cylinder length=0.05 radius=0.1; visual mesh filename=package://bme_ros2_navigation/meshes/wheel.dae scale=1.25 1.25 1.25
- link left_wheel: geometry collision cylinder length=0.05 radius=0.1; visual mesh filename=package://bme_ros2_navigation/meshes/wheel.dae scale=1.25 1.25 1.25
- link right_rear_wheel: geometry collision cylinder length=0.05 radius=0.1; visual mesh filename=package://bme_ros2_navigation/meshes/wheel.dae scale=1.25 1.25 1.25
- link right_wheel: geometry collision cylinder length=0.05 radius=0.1; visual mesh filename=package://bme_ros2_navigation/meshes/wheel.dae scale=1.25 1.25 1.25
